File: pcb/vfd-display-front.kicad_pcb (KiCad board)
At the start: 2 copper layers, 201.9 x 54.6 mm, 61 parts, among them CON1 AVR-ISP-10, IC1 ATMEGA88A-A, IC2 TD62C950RF, IC3 TD62C950RF, J1 HEADER_5, P1 CONN_02X05, P2 CONN_01X03, P3 CONN_01X02, P4 CONN_01X04, P5 CONN_01X02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

Commit message: Fix mess with libraries.
Parts:
- IC2, IC3: footprint TD62C950RF:SSOP60-P-0.65A -> TD62C950RF:TD62C950RF-SSOP60-P-0.65A
