File: pcb/vfd-display-front.sch (KiCad schematic (older format))
At the start: 57 parts, among them CON1 AVR-ISP-10, IC1 ATMEGA88A-A, IC2 TD62C950RF, IC3 TD62C950RF, J1 HEADER_5, P1 CONN_02X05, P2 CONN_01X03, P3 CONN_01X02, P4 CONN_01X04, P5 CONN_01X02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

Commit message: Fix mess with libraries.
Parts:
- IC2, IC3: footprint TD62C950RF:SSOP60-P-0.65A -> TD62C950RF:TD62C950RF-SSOP60-P-0.65A
Changed lines of the file:
@@
 LIBS:contrib
 LIBS:valves
-LIBS:futaba-vfd
 LIBS:w_connectors
 LIBS:w_device
@@
 LIBS:crystal
 LIBS:ESP8266
-LIBS:td62c950rf
+LIBS:futaba-vfd
+LIBS:TD62C950RF
 LIBS:vfd-display-front-cache
 EELAYER 25 0
@@
 F 0 "IC2" H 8500 5150 45  0000 L BNN
 F 1 "TD62C950RF" H 8500 750 45  0000 L BNN
-F 2 "TD62C950RF:SSOP60-P-0.65A" H 8630 3300 20  0001 C CNN
+F 2 "TD62C950RF:TD62C950RF-SSOP60-P-0.65A" H 8630 3300 20  0001 C CNN
 F 3 "" H 8600 3150 60  0001 C CNN
 	1    8600 3150
@@
 F 0 "IC3" H 11500 5150 45  0000 L BNN
 F 1 "TD62C950RF" H 11500 750 45  0000 L BNN
-F 2 "TD62C950RF:SSOP60-P-0.65A" H 11630 3300 20  0001 C CNN
+F 2 "TD62C950RF:TD62C950RF-SSOP60-P-0.65A" H 11630 3300 20  0001 C CNN
 F 3 "" H 11600 3150 60  0001 C CNN
 	1    11600 3150
