File: pcb/vfd-display-front/vfd-display-front.sch (KiCad schematic (older format))
At the start: 57 parts, among them CON1 AVR-ISP-10, IC1 ATMEGA88A-A, IC2 TD62C950RF, IC3 TD62C950RF, J1 HEADER_5, P1 CONN_02X05, P2 CONN_01X03, P3 CONN_01X02, P4 CONN_01X04, P5 CONN_01X02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

Commit message: Add some libraries for Geiger.
Parts:
- L1: symbol INDUCTOR -> INDUCTOR-RESCUE-vfd-display-front
- U3: symbol LM1117-3.3 -> LM1117-3.3-RESCUE-vfd-display-front
Changed lines of the file:
@@
 EESchema Schematic File Version 2
+LIBS:vfd-display-front-rescue
 LIBS:power
 LIBS:device
@@
 $EndComp
 $Comp
-L INDUCTOR L1
+L INDUCTOR-RESCUE-vfd-display-front L1
 U 1 1 578034BB
 P 12550 8100
@@
 $EndComp
 $Comp
-L LM1117-3.3 U3
+L LM1117-3.3-RESCUE-vfd-display-front U3
 U 1 1 578CCB5D
 P 14400 8100
