File: pcb/geiger/geiger.sch (KiCad schematic (older format))
At the start: 18 parts, among them K1 RELAY_DPST, K2 RELAY_DPST, Q1 BC307, Q2 BC140, Q3 BC140, U1 LM208, X1 crystal

Commit message: Add Geiger, transformer models.
Parts:
- added L2: FLYBACK_TRANS, symbol FLYBACK_TRANS
- added V?: EAA91, symbol EAA91
- gave numbers to parts that had none: 1
Changed lines of the file:
@@
 LIBS:lm208
 LIBS:gm_sbm-20
+LIBS:flyback_trans
+LIBS:eaa91
 LIBS:geiger-cache
 EELAYER 25 0
@@
 $EndComp
 $Comp
-L GM_SBM-20 G?
+L GM_SBM-20 G1
 U 1 1 59DBE4B1
 P 9300 3900
-F 0 "G?" H 9350 3940 60  0000 C CNN
+F 0 "G1" H 9350 3940 60  0000 C CNN
 F 1 "GM_SBM-20" H 9570 3720 60  0000 C CNN
 F 2 "" H 9300 3900 60  0001 C CNN
@@
 	1    0    0    -1
 $EndComp
+$Comp
+L FLYBACK_TRANS L2
+U 1 1 59E0D56C
+P 8450 5350
+F 0 "L2" H 8360 5740 60  0000 C CNN
+F 1 "FLYBACK_TRANS" H 8450 5150 28  0000 C CNN
+F 2 "" H 8450 5350 60  0001 C CNN
+F 3 "" H 8450 5350 60  0001 C CNN
+	1    8450 5350
+	1    0    0    -1
+$EndComp
+$Comp
+L EAA91 V?
+U 1 1 59E3E67D
+P 7400 4950
+F 0 "V?" H 7270 5230 60  0000 C CNN
+F 1 "EAA91" H 7590 4850 60  0000 C CNN
+F 2 "" H 7400 4950 60  0001 C CNN
+F 3 "" H 7400 4950 60  0001 C CNN
+	1    7400 4950
+	1    0    0    -1
+$EndComp

Commit message: Add almost complete Geiger schematic (without connections to MCU).
Parts:
- removed L2: FLYBACK_TRANS, symbol FLYBACK_TRANS
- removed V?: EAA91, symbol EAA91
- added C1, C2: 100u, Capacitors_ThroughHole:CP_Radial_D6.3mm_P2.50mm, symbol CP
- added C10: 10n, Capacitors_SMD:C_1206_HandSoldering, symbol C
- added C11: 470n, Capacitors_ThroughHole:C_Rect_L27.0mm_W9.0mm_P23.00mm, symbol C
- added C12, C17, C18, C23, C26, C3, C4, C7: 100n, Capacitors_SMD:C_1206_HandSoldering, symbol C
- added C13, C14, C5, C6: 1000u, Capacitors_ThroughHole:CP_Radial_D16.0mm_P7.50mm, symbol CP
- added C15: 47u, Capacitors_ThroughHole:CP_Radial_D6.3mm_P2.50mm, symbol CP
- added C24: 10n, Capacitors_ThroughHole:C_Disc_D5.1mm_W3.2mm_P5.00mm, symbol C
- added C8: 100n, Capacitors_ThroughHole:C_Rect_L33.0mm_W13.0mm_P27.50mm_MKS4, symbol C
- added C9: 47u, Capacitors_ThroughHole:CP_Radial_D8.0mm_P5.00mm, symbol CP
- added D1, D4: D_Zener, Diodes_ThroughHole:D_DO-41_SOD81_P2.54mm_Vertical_AnodeUp, symbol D_Zener
- added D2, D3: D, Diodes_SMD:D_SMB, symbol D
- added D5, D6: D, Diodes_ThroughHole:D_DO-41_SOD81_P10.16mm_Horizontal, symbol D
- added D7: D_Schottky, Diodes_ThroughHole:D_DO-35_SOD27_P7.62mm_Horizontal, symbol D_Schottky
- added J1, J2, J5: Conn_01x02, Terminal_Blocks:TerminalBlock_Pheonix_MKDS1.5-2pol, symbol Conn_01x02
- added J3: Conn_01x03, Pin_Headers:Pin_Header_Straight_1x03_Pitch2.54mm, symbol Conn_01x03
- added J4: Conn_01x06, Terminal_Blocks:TerminalBlock_Pheonix_PT-3.5mm_6pol, symbol Conn_01x06
- added J6, J7: Conn_02x05_Odd_Even, Pin_Headers:Pin_Header_Straight_2x05_Pitch2.54mm, symbol Conn_02x05_Odd_Even
- added L1: FLYBACK_TRANS, FLYBACK_TRANS:FLYBACK_TRANS, symbol FLYBACK_TRANS
- added Q1: BC107, TO_SOT_Packages_THT:TO-18-3, symbol BC107
- added Q2: BC140, TO_SOT_Packages_THT:TO-39-3, symbol BC140
- added Q3: BC160, TO_SOT_Packages_THT:TO-39-3, symbol BC160
- added Q4: IRF540N, TO_SOT_Packages_THT:TO-220-3_Vertical, symbol IRF540N
- added Q8, Q9: BC847, TO_SOT_Packages_SMD:SOT-23, symbol BC847
- added R1: 1k, Resistors_ThroughHole:R_Axial_DIN0309_L9.0mm_D3.2mm_P12.70mm_Horizontal, symbol R
- added R10: 4k7, Resistors_SMD:R_1206_HandSoldering, symbol R
- added R11, R12, R13, R14, R15, R17, R19, R21, R22, R23, R9: 1M, Resistors_SMD:R_1206_HandSoldering, symbol R
- added R16: 10, Resistors_ThroughHole:R_Axial_DIN0617_L17.0mm_D6.0mm_P30.48mm_Horizontal, symbol R
- added R18, R37, R38: 47k, Resistors_SMD:R_1206_HandSoldering, symbol R
- added R2, R34: 47k, Resistors_ThroughHole:R_Axial_DIN0309_L9.0mm_D3.2mm_P12.70mm_Horizontal, symbol R
- added R20: 330k, Resistors_SMD:R_1206_HandSoldering, symbol R
- added R24: 2k2, Resistors_SMD:R_1206_HandSoldering, symbol R
- added R25, R26: 100k, Resistors_ThroughHole:R_Axial_DIN0411_L9.9mm_D3.6mm_P12.70mm_Horizontal, symbol R
- added R28, R39: 10k, Resistors_ThroughHole:R_Axial_DIN0411_L9.9mm_D3.6mm_P12.70mm_Horizontal, symbol R
- added R29, R32, R35, R36: 10k, Resistors_SMD:R_1206_HandSoldering, symbol R
- added R3: 4k7, Resistors_ThroughHole:R_Axial_DIN0309_L9.0mm_D3.2mm_P12.70mm_Horizontal, symbol R
- added R33: 22k, Resistors_SMD:R_1206_HandSoldering, symbol R
- added R4: 4k7, Resistors_ThroughHole:R_Axial_DIN0411_L9.9mm_D3.6mm_P12.70mm_Horizontal, symbol R
- added R5: 10, Resistors_ThroughHole:R_Axial_DIN0309_L9.0mm_D3.2mm_P12.70mm_Horizontal, symbol R
- added R6: 470, Resistors_ThroughHole:R_Axial_DIN0309_L9.0mm_D3.2mm_P12.70mm_Horizontal, symbol R
- added R7, R8: 1k, Resistors_ThroughHole:R_Axial_DIN0411_L9.9mm_D3.6mm_P12.70mm_Horizontal, symbol R
- added RV1: 100k, Potentiometers:Potentiometer_Trimmer_Bourns_3006P, symbol POT
- added U1: MSP430G2553_PW20, Housings_DIP:DIP-20_W7.62mm_LongPads, symbol MSP430G2553_PW20
- added U2: 74HC595, Housings_DIP:DIP-16_W7.62mm_LongPads, symbol 74HC595
- added U3: AD558, Housings_DIP:DIP-16_W7.62mm_LongPads, symbol AD558
- added V1: EAA91, tube_sockets:HEPTAL1, symbol EAA91
- C16: renamed from C1; footprint (none) -> Capacitors_SMD:C_1206_HandSoldering
- C19: renamed from C2; footprint (none) -> Capacitors_ThroughHole:C_Disc_D5.0mm_W2.5mm_P5.00mm
- C20: renamed from C3; footprint (none) -> Capacitors_ThroughHole:C_Disc_D5.0mm_W2.5mm_P5.00mm
- C21: renamed from C4; footprint (none) -> Capacitors_ThroughHole:C_Disc_D5.0mm_W2.5mm_P5.00mm
- C22: renamed from C5; footprint (none) -> Capacitors_ThroughHole:C_Disc_D5.0mm_W2.5mm_P5.00mm
- C25: renamed from C6; footprint (none) -> Capacitors_ThroughHole:C_Disc_D5.0mm_W2.5mm_P5.00mm
- G1: footprint (none) -> GM_sbm-20:GM_SBM-20
- R27: renamed from R1; footprint (none) -> Resistors_SMD:R_1206_HandSoldering
- R30: renamed from R2; footprint (none) -> Resistors_ThroughHole:R_Axial_DIN0207_L6.3mm_D2.5mm_P10.16mm_Horizontal
- R31: renamed from R3; footprint (none) -> Resistors_ThroughHole:R_Axial_DIN0207_L6.3mm_D2.5mm_P10.16mm_Horizontal
- X1: value crystal -> 5.7MHz
- renumbered L1 to L2, Q2 to Q5, Q3 to Q6, Q1 to Q7, U1 to U4
Connections:
- net labels added: +3.3V, +3V3, -VDC, DAC_CE, DAC_CLK, DAC_CS, DAC_IN, DAC_LATCH, EYE_GRID, EYE_VOL, FLYBACK_PULSE, GM_PULSE, GM_VOL, MCU_CLOCK, REL_HEATER_1, REL_HEATER_2, SCL, SDA
- wire segments 25 -> 315
- no-connect marks 0 -> 10
Other:
- moved on the sheet: C16, C19, C20, C21, C22, C25, K1, K2, L2, Q5, Q6, Q7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
