File: pcb/geiger/geiger.sch (KiCad schematic (older format))
At the start: 100 parts, among them J1 Conn_01x02, J2 Conn_01x02, J3 Conn_01x03, J4 Conn_01x06, J5 Conn_01x02, J6 Conn_02x05_Odd_Even, J7 Conn_02x05_Odd_Even, K1 RELAY_DPST, K2 RELAY_DPST, Q1 BC107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

Commit message: Add board in-process.
Parts:
- removed C1: 100u, Capacitors_ThroughHole:CP_Radial_D6.3mm_P2.50mm, symbol CP
- removed C15: 47u, Capacitors_ThroughHole:CP_Radial_D6.3mm_P2.50mm, symbol CP
- R1, R2, R3, R34, R5: footprint Resistors_ThroughHole:R_Axial_DIN0309_L9.0mm_D3.2mm_P12.70mm_Horizontal -> Resistors_ThroughHole:R_Axial_DIN0207_L6.3mm_D2.5mm_P10.16mm_Horizontal
- R25, R26, R39: footprint Resistors_ThroughHole:R_Axial_DIN0411_L9.9mm_D3.6mm_P12.70mm_Horizontal -> Resistors_ThroughHole:R_Axial_DIN0309_L9.0mm_D3.2mm_P12.70mm_Horizontal
- R28, R4, R7, R8: footprint Resistors_ThroughHole:R_Axial_DIN0411_L9.9mm_D3.6mm_P12.70mm_Horizontal -> Resistors_ThroughHole:R_Axial_DIN0207_L6.3mm_D2.5mm_P10.16mm_Horizontal
Connections:
- net labels added: RST, TEST
- wire segments 315 -> 331
Other:
- moved on the sheet: C12, D2, J3, R6

Commit message: Further pcb changes.
Connections:
- wire segments 331 -> 339
Changed lines of the file:
@@
 L Conn_01x06 J4
 U 1 1 59EA7543
-P 10100 3350
-F 0 "J4" H 10100 3650 50  0000 C CNN
-F 1 "Conn_01x06" H 10100 2950 50  0000 C CNN
-F 2 "Terminal_Blocks:TerminalBlock_Pheonix_PT-3.5mm_6pol" H 10100 3350 50  0001 C CNN
-F 3 "" H 10100 3350 50  0001 C CNN
-	1    10100 3350
-	1    0    0    -1
+P 10100 3450
+F 0 "J4" H 10100 3750 50  0000 C CNN
+F 1 "Conn_01x06" H 10100 3050 50  0000 C CNN
+F 2 "Terminal_Blocks:TerminalBlock_Pheonix_PT-3.5mm_6pol" H 10100 3450 50  0001 C CNN
+F 3 "" H 10100 3450 50  0001 C CNN
+	1    10100 3450
+	1    0    0    1
 $EndComp
 $Comp
@@
 L Conn_01x02 J5
 U 1 1 59EA89A8
-P 10100 4050
-F 0 "J5" H 10100 4150 50  0000 C CNN
-F 1 "Conn_01x02" H 10100 3850 50  0000 C CNN
-F 2 "Terminal_Blocks:TerminalBlock_Pheonix_MKDS1.5-2pol" H 10100 4050 50  0001 C CNN
-F 3 "" H 10100 4050 50  0001 C CNN
-	1    10100 4050
-	1    0    0    -1
+P 10100 4150
+F 0 "J5" H 10100 4250 50  0000 C CNN
+F 1 "Conn_01x02" H 10100 3950 50  0000 C CNN
+F 2 "Terminal_Blocks:TerminalBlock_Pheonix_MKDS1.5-2pol" H 10100 4150 50  0001 C CNN
+F 3 "" H 10100 4150 50  0001 C CNN
+	1    10100 4150
+	1    0    0    1
 $EndComp
 NoConn ~ 8300 2800
@@
 	4750 2800 5650 2800
 Wire Wire Line
-	6500 2650 4750 2650
-Wire Wire Line
 	6750 3750 6900 3750
 Wire Wire Line
 	6850 3750 6850 4000
 Wire Wire Line
-	5900 2900 6500 2900
-Wire Wire Line
 	7700 4000 7650 4000
 Wire Wire Line
-	7700 2900 7700 4000
+	7700 2800 7700 4000
 Wire Wire Line
 	7700 3750 7650 3750
-Wire Wire Line
-	7700 2900 7250 2900
 Connection ~ 7700 3750
 Wire Wire Line
@@
 Connection ~ 6850 3750
 Wire Wire Line
-	5900 2900 5900 5550
+	5900 2550 5900 5550
 Connection ~ 6250 3050
 Wire Wire Line
@@
 	8650 2950 8650 2650
 Wire Wire Line
-	8650 2650 7250 2650
-Wire Wire Line
 	8000 2950 7950 2950
 Wire Wire Line
@@
 Connection ~ 8700 3250
 Wire Wire Line
-	9150 3150 9900 3150
-Wire Wire Line
-	9900 3250 9550 3250
-Wire Wire Line
-	9900 3450 9500 3450
-Wire Wire Line
 	9500 3450 9500 3700
 Wire Wire Line
@@
 	9400 3500 9400 3350
 Wire Wire Line
-	9400 3350 9900 3350
-Wire Wire Line
-	9900 4050 9850 4050
-Wire Wire Line
 	9850 4050 9850 3650
 Wire Wire Line
-	9850 3650 9900 3650
-Wire Wire Line
-	9900 3550 9750 3550
-Wire Wire Line
 	9750 3550 9750 3600
 Wire Wire Line
@@
 Wire Wire Line
 	9550 5550 9550 4150
-Wire Wire Line
-	9550 4150 9900 4150
 Connection ~ 5900 3750
 Connection ~ 4850 3750
@@
 Wire Wire Line
 	4850 3650 4850 3900
+Wire Wire Line
+	4750 2650 6050 2650
+Wire Wire Line
+	6050 2650 6050 2900
+Wire Wire Line
+	6050 2900 6500 2900
+Wire Wire Line
+	7250 2900 7500 2900
+Wire Wire Line
+	7500 2900 7500 2650
+Wire Wire Line
+	7500 2650 8650 2650
+Wire Wire Line
+	7700 2800 7300 2800
+Wire Wire Line
+	7300 2800 7300 2650
+Wire Wire Line
+	7300 2650 7250 2650
+Wire Wire Line
+	5900 2550 6400 2550
+Wire Wire Line
+	6400 2550 6400 2650
+Wire Wire Line
+	6400 2650 6500 2650
+Wire Wire Line
+	9900 4050 9850 4050
+Wire Wire Line
+	9550 4150 9900 4150
+Wire Wire Line
+	9850 3650 9900 3650
+Wire Wire Line
+	9750 3550 9900 3550
+Wire Wire Line
+	9500 3450 9900 3450
+Wire Wire Line
+	9400 3350 9900 3350
+Wire Wire Line
+	9900 3250 9550 3250
+Wire Wire Line
+	9900 3150 9150 3150
 $EndSCHEMATC

Commit message: Finish Geiger schematic.
Parts:
- added C1, C15, C27: 33n, Capacitors_ThroughHole:C_Disc_D5.0mm_W2.5mm_P5.00mm, symbol C
- C13: value 1000u -> 220u; footprint Capacitors_ThroughHole:CP_Radial_D16.0mm_P7.50mm -> Capacitors_ThroughHole:CP_Radial_D8.0mm_P5.00mm
- C25: value 1n -> 33n
Connections:
- wire segments 339 -> 357
- no-connect marks 10 -> 12
Other:
- moved on the sheet: C22, C25, D6, R37
Changed lines of the file:
@@
 L C C22
 U 1 1 59C98628
-P 14200 5050
-F 0 "C22" H 14225 5150 50  0000 L CNN
-F 1 "47p" H 14225 4950 50  0000 L CNN
-F 2 "Capacitors_ThroughHole:C_Disc_D5.0mm_W2.5mm_P5.00mm" H 14238 4900 50  0001 C CNN
-F 3 "" H 14200 5050 50  0000 C CNN
-	1    14200 5050
+P 14150 5050
+F 0 "C22" H 14175 5150 50  0000 L CNN
+F 1 "47p" H 14175 4950 50  0000 L CNN
+F 2 "Capacitors_ThroughHole:C_Disc_D5.0mm_W2.5mm_P5.00mm" H 14188 4900 50  0001 C CNN
+F 3 "" H 14150 5050 50  0000 C CNN
+	1    14150 5050
 	-1   0    0    1
 $EndComp
@@
 L C C25
 U 1 1 59C9869E
-P 14700 5250
-F 0 "C25" H 14725 5350 50  0000 L CNN
-F 1 "1n" H 14725 5150 50  0000 L CNN
-F 2 "Capacitors_ThroughHole:C_Disc_D5.0mm_W2.5mm_P5.00mm" H 14738 5100 50  0001 C CNN
-F 3 "" H 14700 5250 50  0000 C CNN
-	1    14700 5250
-	0    -1   -1   0
+P 14450 5050
+F 0 "C25" H 14475 5150 50  0000 L CNN
+F 1 "33n" H 14475 4950 50  0000 L CNN
+F 2 "Capacitors_ThroughHole:C_Disc_D5.0mm_W2.5mm_P5.00mm" H 14488 4900 50  0001 C CNN
+F 3 "" H 14450 5050 50  0000 C CNN
+	1    14450 5050
+	1    0    0    -1
 $EndComp
 $Comp
@@
 L D D6
 U 1 1 59E6BA55
-P 6600 4350
-F 0 "D6" H 6600 4450 50  0000 C CNN
-F 1 "D" H 6600 4250 50  0000 C CNN
-F 2 "Diodes_ThroughHole:D_DO-41_SOD81_P10.16mm_Horizontal" H 6600 4350 50  0001 C CNN
-F 3 "" H 6600 4350 50  0001 C CNN
-	1    6600 4350
+P 6600 4450
+F 0 "D6" H 6600 4550 50  0000 C CNN
+F 1 "D" H 6600 4350 50  0000 C CNN
+F 2 "Diodes_ThroughHole:D_DO-41_SOD81_P10.16mm_Horizontal" H 6600 4450 50  0001 C CNN
+F 3 "" H 6600 4450 50  0001 C CNN
+	1    6600 4450
 	0    1    1    0
 $EndComp
@@
 L GND #PWR032
 U 1 1 59EA857C
-P 9500 3700
-F 0 "#PWR032" H 9500 3450 50  0001 C CNN
-F 1 "GND" H 9500 3550 50  0000 C CNN
-F 2 "" H 9500 3700 50  0001 C CNN
-F 3 "" H 9500 3700 50  0001 C CNN
-	1    9500 3700
-	1    0    0    -1
-$EndComp
-Text GLabel 9350 3500 0    60   Input ~ 0
+P 9650 3700
+F 0 "#PWR032" H 9650 3450 50  0001 C CNN
+F 1 "GND" H 9650 3550 50  0000 C CNN
+F 2 "" H 9650 3700 50  0001 C CNN
+F 3 "" H 9650 3700 50  0001 C CNN
+	1    9650 3700
+	1    0    0    -1
+$EndComp
+Text GLabel 9550 3450 0    60   Input ~ 0
 EYE_GRID
 $Comp
@@
 F 3 "" H 14800 9200 50  0001 C CNN
 	1    14800 9200
-	0    -1   -1   0
+	0    1    -1   0
 $EndComp
 $Comp
@@
 L R R37
 U 1 1 59F01610
-P 15150 5550
-F 0 "R37" V 15230 5550 50  0000 C CNN
-F 1 "47k" V 15150 5550 50  0000 C CNN
-F 2 "Resistors_SMD:R_1206_HandSoldering" V 15080 5550 50  0001 C CNN
-F 3 "" H 15150 5550 50  0001 C CNN
-	1    15150 5550
+P 15550 5000
+F 0 "R37" V 15630 5000 50  0000 C CNN
+F 1 "47k" V 15550 5000 50  0000 C CNN
+F 2 "Resistors_SMD:R_1206_HandSoldering" V 15480 5000 50  0001 C CNN
+F 3 "" H 15550 5000 50  0001 C CNN
+	1    15550 5000
 	-1   0    0    1
 $EndComp
@@
 L +3V3 #PWR040
 U 1 1 59F0414D
-P 15150 5250
-F 0 "#PWR040" H 15150 5100 50  0001 C CNN
-F 1 "+3V3" H 15150 5390 50  0000 C CNN
-F 2 "" H 15150 5250 50  0001 C CNN
-F 3 "" H 15150 5250 50  0001 C CNN
-	1    15150 5250
+P 15550 4750
+F 0 "#PWR040" H 15550 4600 50  0001 C CNN
+F 1 "+3V3" H 15550 4890 50  0000 C CNN
+F 2 "" H 15550 4750 50  0001 C CNN
+F 3 "" H 15550 4750 50  0001 C CNN
+	1    15550 4750
 	1    0    0    -1
 $EndComp
@@
 P 11900 3000
 F 0 "C13" H 11925 3100 50  0000 L CNN
-F 1 "1000u" H 11925 2900 50  0000 L CNN
-F 2 "Capacitors_ThroughHole:CP_Radial_D16.0mm_P7.50mm" H 11938 2850 50  0001 C CNN
+F 1 "220u" H 11925 2900 50  0000 L CNN
+F 2 "Capacitors_ThroughHole:CP_Radial_D8.0mm_P5.00mm" H 11938 2850 50  0001 C CNN
 F 3 "" H 11900 3000 50  0001 C CNN
 	1    11900 3000
@@
 	13800 4500 13800 4650
 Wire Wire Line
-	13400 4600 14200 4600
+	13400 4600 14150 4600
 Wire Wire Line
 	13400 4600 13400 4500
@@
 	13800 5250 13800 5050
 Wire Wire Line
-	12800 5250 14550 5250
-Wire Wire Line
 	13150 5200 13150 5250
 Connection ~ 13150 5250
 Wire Wire Line
-	13550 5300 13550 5250
+	13550 5250 13550 5300
 Connection ~ 13550 5250
 Wire Wire Line
-	14200 4600 14200 4900
+	14150 4600 14150 4900
 Connection ~ 13800 5250
 Wire Wire Line
-	14200 5200 14200 5250
-Connection ~ 14200 5250
+	14150 5250 14150 5200
+Connection ~ 14150 5250
 Wire Wire Line
 	13000 5650 13000 5800
@@
 	5900 2550 5900 5550
 Connection ~ 6250 3050
-Wire Wire Line
-	6900 4150 6600 4150
-Wire Wire Line
-	6600 4050 6600 4200
-Connection ~ 6600 4150
-Wire Wire Line
-	6900 4250 6900 4800
-Wire Wire Line
-	6900 4550 6600 4550
-Wire Wire Line
-	6600 4550 6600 4500
-Connection ~ 6900 4550
 Connection ~ 6250 3450
 Wire Wire Line
@@
 Connection ~ 8700 3250
 Wire Wire Line
-	9500 3450 9500 3700
-Wire Wire Line
-	9350 3500 9400 3500
-Wire Wire Line
-	9400 3500 9400 3350
-Wire Wire Line
 	9850 4050 9850 3650
 Wire Wire Line
-	9750 3550 9750 3600
-Wire Wire Line
-	9750 3600 8350 3600
-Wire Wire Line
-	8350 3600 8350 3300
+	8350 3550 8350 3300
 Wire Wire Line
 	5900 5550 9550 5550
@@
 Connection ~ 13650 8500
 Wire Wire Line
-	14800 9050 14800 9000
-Wire Wire Line
-	14800 9000 15000 9000
+	15000 9000 14800 9000
 Wire Wire Line
 	15000 8400 15000 9200
-Wire Wire Line
-	15000 9200 14950 9200
 Wire Wire Line
 	14750 8850 15000 8850
@@
 Connection ~ 14250 8950
 Wire Wire Line
-	14600 9200 14650 9200
-Wire Wire Line
 	15350 8400 15400 8400
 Connection ~ 15000 8400
 Wire Wire Line
-	14850 5250 14900 5250
-Wire Wire Line
-	14900 5250 14900 5750
-Wire Wire Line
-	14900 5750 15150 5750
-Wire Wire Line
-	15150 5700 15150 5900
-Connection ~ 15150 5750
-Wire Wire Line
 	15150 6250 15150 6200
 Wire Wire Line
-	15300 5850 15150 5850
-Connection ~ 15150 5850
-Wire Wire Line
-	15150 5400 15150 5250
+	15550 4850 15550 4750
 Wire Wire Line
 	1600 9300 2250 9300
@@
 	9850 3650 9900 3650
 Wire Wire Line
-	9750 3550 9900 3550
-Wire Wire Line
-	9500 3450 9900 3450
-Wire Wire Line
-	9400 3350 9900 3350
-Wire Wire Line
 	9900 3250 9550 3250
 Wire Wire Line
 	9900 3150 9150 3150
+$Comp
+L C C1
+U 1 1 5A064247
+P 14700 5050
+F 0 "C1" H 14725 5150 50  0000 L CNN
+F 1 "33n" H 14725 4950 50  0000 L CNN
+F 2 "Capacitors_ThroughHole:C_Disc_D5.0mm_W2.5mm_P5.00mm" H 14738 4900 50  0001 C CNN
+F 3 "" H 14700 5050 50  0000 C CNN
+	1    14700 5050
+	1    0    0    -1
+$EndComp
+$Comp
+L C C15
+U 1 1 5A066A8F
+P 14950 5050
+F 0 "C15" H 14975 5150 50  0000 L CNN
+F 1 "33n" H 14975 4950 50  0000 L CNN
+F 2 "Capacitors_ThroughHole:C_Disc_D5.0mm_W2.5mm_P5.00mm" H 14988 4900 50  0001 C CNN
+F 3 "" H 14950 5050 50  0000 C CNN
+	1    14950 5050
+	1    0    0    -1
+$EndComp
+Wire Wire Line
+	15550 5150 15550 5550
+Wire Wire Line
+	15550 5550 15150 5550
+Wire Wire Line
+	15150 5550 15150 5900
+Wire Wire Line
+	15300 5850 15150 5850
+Connection ~ 15150 5850
+Connection ~ 15550 5250
+$Comp
+L C C27
+U 1 1 5A069169
+P 15200 5050
+F 0 "C27" H 15225 5150 50  0000 L CNN
+F 1 "33n" H 15225 4950 50  0000 L CNN
+F 2 "Capacitors_ThroughHole:C_Disc_D5.0mm_W2.5mm_P5.00mm" H 15238 4900 50  0001 C CNN
+F 3 "" H 15200 5050 50  0000 C CNN
+	1    15200 5050
+	1    0    0    -1
+$EndComp
+Wire Wire Line
+	12800 5250 14450 5250
+Wire Wire Line
+	14450 5250 14450 5200
+Wire Wire Line
+	14450 4900 14450 4850
+Wire Wire Line
+	14450 4850 14700 4850
+Wire Wire Line
+	14700 4850 14700 4900
+Wire Wire Line
+	14700 5200 14700 5250
+Wire Wire Line
+	14700 5250 14950 5250
+Wire Wire Line
+	14950 5250 14950 5200
+Wire Wire Line
+	14950 4900 14950 4850
+Wire Wire Line
+	14950 4850 15200 4850
+Wire Wire Line
+	15200 4850 15200 4900
+Wire Wire Line
+	15200 5200 15200 5250
+Wire Wire Line
+	15200 5250 15550 5250
+Wire Wire Line
+	14800 9000 14800 9050
+Wire Wire Line
+	14650 9200 14600 9200
+Wire Wire Line
+	15000 9200 14950 9200
+Wire Wire Line
+	9900 3550 9650 3550
+Wire Wire Line
+	9650 3550 9650 3700
+Wire Wire Line
+	9900 3350 8800 3350
+Wire Wire Line
+	8800 3350 8800 3550
+Wire Wire Line
+	8800 3550 8350 3550
+Wire Wire Line
+	9900 3450 9550 3450
+Text GLabel 6450 8200 2    60   Input ~ 0
+GM_PULSE
+Wire Wire Line
+	6450 8200 6300 8200
+Wire Wire Line
+	6300 8200 6300 8400
+Wire Wire Line
+	6300 8400 6150 8400
+Text GLabel 2100 8600 0    60   Input ~ 0
+FLYBACK_PULSE
+Wire Wire Line
+	2250 8600 2100 8600
+Wire Wire Line
+	6600 4050 6600 4300
+Wire Wire Line
+	6900 4150 6800 4150
+Wire Wire Line
+	6800 4150 6800 4600
+Wire Wire Line
+	6600 4600 6900 4600
+Wire Wire Line
+	6900 4600 6900 4800
+Connection ~ 6800 4600
+Wire Wire Line
+	6900 4250 6600 4250
+Connection ~ 6600 4250
+Text GLabel 2100 8900 0    60   Input ~ 0
+GM_VOL
+Text GLabel 2100 8800 0    60   Input ~ 0
+EYE_VOL
+Wire Wire Line
+	2250 8900 2100 8900
+Wire Wire Line
+	2250 8800 2100 8800
+Text GLabel 2100 8700 0    60   Input ~ 0
+REL_HEATER_2
+Wire Wire Line
+	2250 8700 2100 8700
+Text GLabel 2100 8500 0    60   Input ~ 0
+REL_HEATER_1
+Wire Wire Line
+	2250 8500 2100 8500
+NoConn ~ 2250 8400
+NoConn ~ 6150 9150
 $EndSCHEMATC

Commit message: Finish Geiger board.
Parts:
- removed C17: 100n, Capacitors_SMD:C_1206_HandSoldering, symbol C
- removed R17: 1M, Resistors_SMD:R_1206_HandSoldering, symbol R
- C13: footprint Capacitors_ThroughHole:CP_Radial_D8.0mm_P5.00mm -> Capacitors_ThroughHole:CP_Radial_D12.5mm_P5.00mm
- C14: value 1000u -> 220u; footprint Capacitors_ThroughHole:CP_Radial_D16.0mm_P7.50mm -> Capacitors_ThroughHole:CP_Radial_D12.5mm_P5.00mm
- D5, D6: footprint Diodes_ThroughHole:D_DO-41_SOD81_P10.16mm_Horizontal -> Diodes_ThroughHole:D_DO-41_SOD81_P12.70mm_Horizontal
- D7: footprint Diodes_ThroughHole:D_DO-35_SOD27_P7.62mm_Horizontal -> Diodes_ThroughHole:D_DO-35_SOD27_P10.16mm_Horizontal
- R12: footprint Resistors_SMD:R_1206_HandSoldering -> Resistors_ThroughHole:R_Axial_DIN0309_L9.0mm_D3.2mm_P12.70mm_Horizontal
- R15: value 1M -> 2M2; footprint Resistors_SMD:R_1206_HandSoldering -> Resistors_ThroughHole:R_Axial_DIN0309_L9.0mm_D3.2mm_P12.70mm_Horizontal
- R25, R26: footprint Resistors_ThroughHole:R_Axial_DIN0309_L9.0mm_D3.2mm_P12.70mm_Horizontal -> Resistors_ThroughHole:R_Axial_DIN0309_L9.0mm_D3.2mm_P15.24mm_Horizontal
Connections:
- wire segments 357 -> 354
Other:
- moved on the sheet: R12, R15

Commit message: Update element values on the schematic.
Parts:
- C1, C15, C27: value 33n -> 47n
- C10: value 10n -> 1n
- C20, C21: value C -> 33p
- C22: value 47p -> 150p
- C25: value 33n -> 22n
- Q2: value BC140 -> BC211
- Q3: value BC160 -> BC313
- R1: value 1k -> 1k5
- R10: value 4k7 -> 3k9
- R11, R13, R14, R21, R22, R23, R9: value 1M -> 180k
- R18, R27, R37, R38: value 47k -> 38k
- R2: value 47k -> 56k
- R20: value 330k -> 475k
- R24: value 2k2 -> 4k7
- R3: value 4k7 -> 3k3
- R39: value 10k -> 6k8
- R5: value 10 -> 1R7

Commit message: Separate some code in Geiger to common module. Add unit test harness. Create unit test for eye.
Parts:
- C24: value 10n -> 33n
- R12: value 1M -> 1M6
- R15: value 2M2 -> 1M6
- R25: value 100k -> 510k
- R26: value 100k -> 10k
Connections:
- net labels added: EYE_ANODE, EYE_SCREEN
- wire segments 354 -> 431
Other:
- moved on the sheet: J4, J5

Commit message: Add new libraries for new Geiger board.
Parts:
- removed D5: D, Diodes_ThroughHole:D_DO-41_SOD81_P12.70mm_Horizontal, symbol D
- removed K2: RELAY_DPST, RELAY_DPST_Telfa_K-8:RELAY_DPST_Telfa_K-8, symbol RELAY_DPST
- removed L1: FLYBACK_TRANS, FLYBACK_TRANS:FLYBACK_TRANS, symbol FLYBACK_TRANS
- removed Q1: BC107, TO_SOT_Packages_THT:TO-18-3, symbol BC107
- removed Q2: BC211, TO_SOT_Packages_THT:TO-39-3, symbol BC140
- removed Q3: BC313, TO_SOT_Packages_THT:TO-39-3, symbol BC160
- removed Q5, Q6: BC140, TO_SOT_Packages_THT:TO-39-3, symbol BC140
- removed U4: LM208, TO-5:TO-5-8_H08C, symbol LM208
- added C17, C33, C34: 10n, Capacitors_SMD:C_1206_HandSoldering, symbol C
- added C28: 22u, Capacitors_Tantalum_SMD:CP_Tantalum_Case-B_EIA-3528-21_Hand, symbol CP
- added C29, C30, C31, C32, C36, C37: 100n, Capacitors_SMD:C_1206_HandSoldering, symbol C
- added C35: 33p, Capacitors_ThroughHole:C_Disc_D5.0mm_W2.5mm_P5.00mm, symbol C
- added D5: SS34, Diodes_SMD:D_SMA-SMB_Universal_Handsoldering, symbol D_Schottky
- added D8: D, Diodes_ThroughHole:D_DO-41_SOD81_P12.70mm_Horizontal, symbol D
- added JP1: Jumper, Pin_Headers:Pin_Header_Straight_1x02_Pitch2.54mm, symbol Jumper
- added L1: L_Core_Ferrite, Choke_SMD:Choke_SMD_12x12mm_h8mm, symbol L_Core_Ferrite
- added L3: L_Core_Ferrite, F1001:F1001_coil, symbol L_Core_Ferrite
- added Q1: BC140, TO_SOT_Packages_THT:TO-39-3, symbol BC140
- added Q2: BC107, TO_SOT_Packages_THT:TO-18-3, symbol BC107
- added Q3: BC211, TO_SOT_Packages_THT:TO-39-3, symbol BC140
- added Q5: BC313, TO_SOT_Packages_THT:TO-39-3, symbol BC160
- added Q6: IRF540N, TO_SOT_Packages_THT:TO-220-3_Vertical, symbol IRF540N
- added R17: 56k, Resistors_ThroughHole:R_Axial_DIN0207_L6.3mm_D2.5mm_P10.16mm_Horizontal, symbol R
- added R40: 3k3, Resistors_ThroughHole:R_Axial_DIN0207_L6.3mm_D2.5mm_P10.16mm_Horizontal, symbol R
- added R41: 1R7, Resistors_ThroughHole:R_Axial_DIN0207_L6.3mm_D2.5mm_P10.16mm_Horizontal, symbol R
- added T1: Transformer_1P_1S, F1001:F1001_trans, symbol Transformer_1P_1S
- added U4: MAA725, TO-5:TO-5-8_H08C, symbol MAA725
- added U5: LM2596, TO_SOT_Packages_SMD:TO-263-5_TabPin3, symbol LM2596
- added U6: MCP1402, TO_SOT_Packages_SMD:SOT-23-5_HandSoldering, symbol MCP1402
- C10: footprint Capacitors_SMD:C_1206_HandSoldering -> Capacitors_SMD:C_0805_HandSoldering
- C11: value 470n -> 2u2; footprint Capacitors_ThroughHole:C_Rect_L27.0mm_W9.0mm_P23.00mm -> Capacitors_ThroughHole:C_Rect_L33.0mm_W13.0mm_P27.50mm_MKS4
- C13, C14: footprint Capacitors_ThroughHole:CP_Radial_D12.5mm_P5.00mm -> Capacitors_ThroughHole:CP_Radial_D13.0mm_P5.00mm
- C2: value 100u -> 4u7
- C24: footprint Capacitors_ThroughHole:C_Disc_D5.1mm_W3.2mm_P5.00mm -> Capacitors_ThroughHole:C_Disc_D11.0mm_W5.0mm_P5.00mm
- C9: value 47u -> 6u8; footprint Capacitors_ThroughHole:CP_Radial_D8.0mm_P5.00mm -> Capacitors_Tantalum_SMD:CP_Tantalum_Case-D_EIA-7343-31_Hand
- L2: footprint L_7x7:L_7x7 -> L_7x7:L_7x7_II
- R1: value 1k5 -> 1k
- R16: value 10 -> 1k5; footprint Resistors_ThroughHole:R_Axial_DIN0617_L17.0mm_D6.0mm_P30.48mm_Horizontal -> Resistors_ThroughHole:R_Axial_DIN0207_L6.3mm_D2.5mm_P10.16mm_Horizontal
- R2: value 56k -> 3k9; footprint Resistors_ThroughHole:R_Axial_DIN0207_L6.3mm_D2.5mm_P10.16mm_Horizontal -> Resistors_SMD:R_1206_HandSoldering
- R21, R22, R23: footprint Resistors_SMD:R_1206_HandSoldering -> Resistors_SMD:R_0805_HandSoldering
- R3: value 3k3 -> 3k9; footprint Resistors_ThroughHole:R_Axial_DIN0207_L6.3mm_D2.5mm_P10.16mm_Horizontal -> Resistors_SMD:R_1206_HandSoldering
- R34: value 47k -> 22k
- R5: value 1R7 -> 3k9; footprint Resistors_ThroughHole:R_Axial_DIN0207_L6.3mm_D2.5mm_P10.16mm_Horizontal -> Resistors_SMD:R_1206_HandSoldering
- R8: value 1k -> 10; footprint Resistors_ThroughHole:R_Axial_DIN0207_L6.3mm_D2.5mm_P10.16mm_Horizontal -> Resistors_ThroughHole:R_Axial_DIN0617_L17.0mm_D6.0mm_P30.48mm_Horizontal
Connections:
- net labels added: +15V, +36V, EYE_PWM, GM_PWM, HEATER1, HEATER2, HEATER_6_3V
- wire segments 431 -> 405
Other:
- moved on the sheet: C1, C11, C13, C14, C15, C16, C19, C2, C20, C21, C22, C23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

Commit message: Add ready schematic and all connections on board.
Parts:
- added C38: 22u, Capacitors_Tantalum_SMD:CP_Tantalum_Case-B_EIA-3528-21_Hand, symbol CP
- added R42: 100, Resistors_ThroughHole:R_Axial_DIN0309_L9.0mm_D3.2mm_P12.70mm_Horizontal, symbol R
- C34: footprint Capacitors_SMD:C_1206_HandSoldering -> Capacitors_ThroughHole:C_Rect_L9.0mm_W3.2mm_P7.50mm_MKT
- C35: footprint Capacitors_ThroughHole:C_Disc_D5.0mm_W2.5mm_P5.00mm -> Capacitors_ThroughHole:C_Rect_L9.0mm_W3.2mm_P7.50mm_MKT
- R1: footprint Resistors_ThroughHole:R_Axial_DIN0207_L6.3mm_D2.5mm_P10.16mm_Horizontal -> Resistors_ThroughHole:R_Axial_DIN0411_L9.9mm_D3.6mm_P12.70mm_Horizontal
- R19: footprint Resistors_SMD:R_1206_HandSoldering -> Resistors_ThroughHole:R_Axial_DIN0309_L9.0mm_D3.2mm_P12.70mm_Horizontal
Connections:
- net DAC_CE is gone; now on net EYE_PWM: U1.9 (P2.1/TA1.1)
- net DAC_CS is gone; now on net GM_PULSE: U1.10 (P2.2/TA1.1)
- net FLYBACK_PULSE is gone; now on net GM_PWM: U1.4 (P1.2/TA0.1/UCA0TXD/PUCA0SIMO/A2/CA2)
- net REL_HEATER_1 is gone; now on net GM_VOL: U1.3 (P1.1/TA0.0/UCA0RXD/UCA0SOMI/A1/CA1)
- net REL_HEATER_2 is gone; now on net HEATER1: U1.5 (P1.3/ADC10CLK/CAOUT/VREF-/VEREF-/A3/CA3)
- net +15V: now also C38.1
- net +3V3: now also C34.2, C35.1
- net +5V: now also K1.2; no longer K1.1
- net -VDC: now also C36.2
- net EYE_GRID: now also J4.6 (Pin_6); no longer J4.3 (Pin_3)
- net EYE_VOL: now also U1.7 (P1.5/TA0.0/UCB0CLK/UCA0STE/A5/CA5/TMS); no longer U1.6 (P1.4/SMCLK/UCB0STE/UCA0CLK/VREF+/VEREF+/A4/CA4/TCK)
- net GM_PULSE: now also C35.2; no longer C35.1, U1.8 (P2.0/TA1.0)
- net GM_PWM: now also R42.1; no longer U6.3 (IN)
- net GM_VOL: no longer U1.7 (P1.5/TA0.0/UCB0CLK/UCA0STE/A5/CA5/TMS)
- net GND: now also J5.2 (Pin_2), T1.4 (SB), C38.2; no longer C34.2, C35.2, C36.2, J5.1 (Pin_1), T1.3 (SA)
- net HEATER2: now also U1.6 (P1.4/SMCLK/UCB0STE/UCA0CLK/VREF+/VEREF+/A4/CA4/TCK)
- net HEATER_6_3V: now also J4.1 (Pin_1), J5.1 (Pin_1), K1.6, K1.8; no longer J5.2 (Pin_2), K1.5, K1.7
- net at D2.1 (K): now also T1.3 (SA); no longer T1.4 (SB)
- net at C11.1, R21.2, R26.1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: now also R25.2; no longer R25.1
- net at J4.4 (Pin_4): now also R26.2
- net at C17.1, C28.1, C29.1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: now also K1.5, K1.7; no longer K1.6, K1.8
- net at D6.1 (K), D8.2 (A), JP1.2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: now also K1.1; no longer K1.2
- removed net EYE_ANODE: J4.6 (Pin_6), R25.2
- net EYE_SCREEN: no longer names the net of J4.5 (Pin_5)
- net EYE_SCREEN: no longer R26.2
- new net: J4.3 (Pin_3), R25.1
- new net: R42.2, U6.3 (IN)
- no-connect marks 12 -> 14
Other:
- moved on the sheet: C23, C30, C31, C32, C35, C36, D2, D7, D8, J4, J5, Q2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
