File: pcb/geiger/geiger.kicad_pcb (KiCad board)
At the start: 2 copper layers, 154.9 x 56.5 mm, 99 parts, among them J1 Conn_01x02, J2 Conn_01x02, J3 Conn_01x03, J4 Conn_01x06, J5 Conn_01x02, J6 Conn_02x05_Odd_Even, J7 Conn_02x05_Odd_Even, K1 RELAY_DPST, K2 RELAY_DPST, Q1 BC107, Q2 BC140, Q3 BC160, Q4 IRF540N, Q5 BC140, Q6 BC140, Q7 BC307, Q8 BC847, Q9 BC847, U1 MSP430G2553_PW20, U2 74HC595, U3 AD558, U4 LM208, X1 5.7MHz

Commit message: Further pcb changes.
Parts:
- added REF**: 1pin, Connect:1pin, F.Cu at (23.5, 87.0)
- added REF**: 1pin, Connect:1pin, F.Cu at (173.4, 87.0)
- added REF**: 1pin, Connect:1pin, F.Cu at (173.4, 186.7)
- C4, C7, D3, R10: moved to B.Cu
- moved C5 378.2 mm to (158.8, 126.4), turned to 180 degrees
- moved C6 366.2 mm to (158.8, 108.0), turned to 180 degrees
- moved C8 341.3 mm to (134.6, 88.9)
- moved D1 339.6 mm to (174.6, 174.0), turned to 180 degrees
- moved R12 329.3 mm to (125.7, 83.8), turned to 180 degrees
- moved D3 317.5 mm to (111.1, 111.8), turned to 180 degrees
- moved R16 274.9 mm to (95.9, 88.9)
- moved K2 251.6 mm to (71.1, 113.7)
- moved D6 251.0 mm to (57.8, 111.1)
- moved R15 240.8 mm to (36.8, 74.3)
- moved R20 236.9 mm to (137.8, 94.6)
- moved R19 234.5 mm to (134.6, 102.9), turned to 90 degrees
- moved R17 230.2 mm to (27.9, 73.7), turned to 270 degrees
- moved Q6 226.3 mm to (25.4, 127.0), turned to 270 degrees
- moved R9 222.4 mm to (48.3, 83.2)
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Connections:
- J4 pad 3: EYE_GRID -> GND
- J4 pad 4: GND -> EYE_GRID
- J5 pad 1: Net-(J4-Pad6) -> Net-(J5-Pad1)
- J5 pad 2: Net-(J5-Pad2) -> Net-(J4-Pad1)
- K1 pad 6: Net-(J5-Pad2) -> Net-(K1-Pad6)
- K1 pad 8: Net-(K1-Pad8) -> Net-(J5-Pad1)
- K2 pad 5: Net-(K1-Pad5) -> Net-(K1-Pad7)
- K2 pad 7: Net-(K1-Pad5) -> Net-(K1-Pad7)
- L1 pad 5: Net-(K1-Pad8) -> Net-(K1-Pad6)
- R16 pad 1: Net-(J5-Pad2) -> Net-(J5-Pad1)
- R25 pad 2: Net-(J4-Pad1) -> Net-(J4-Pad6)
- R26 pad 2: Net-(J4-Pad2) -> Net-(J4-Pad5)
- V1 pad 2: Net-(K1-Pad7) -> Net-(K1-Pad5)
- V1 pad 3: Net-(K1-Pad5) -> Net-(K1-Pad7)
- V1 pad 4: Net-(J4-Pad5) -> Net-(J4-Pad2)
- V1 pad 7: Net-(K1-Pad7) -> Net-(K1-Pad5)
Routing:
- net GND: track 92.1 -> 166.1 mm
- net Net-(L1-Pad2): track 0.00 -> 40.9 mm
- net Net-(Q2-Pad1): track 0.00 -> 18.6 mm
Other:
- board size 154.9 x 56.5 mm -> 162.6 x 112.4 mm

Commit message: Finish Geiger schematic.
Parts:
- added C1: 33n, Capacitors_ThroughHole:C_Disc_D5.0mm_W2.5mm_P5.00mm, F.Cu at (116.2, 173.4)
- added C15: 33n, Capacitors_ThroughHole:C_Disc_D5.0mm_W2.5mm_P5.00mm, F.Cu at (124.5, 178.4)
- added C27: 33n, Capacitors_ThroughHole:C_Disc_D5.0mm_W2.5mm_P5.00mm, F.Cu at (127.6, 178.4)
- C13: value 1000u -> 220u; footprint Capacitors_ThroughHole:CP_Radial_D16.0mm_P7.50mm -> Capacitors_ThroughHole:CP_Radial_D8.0mm_P5.00mm
- C25: value 1n -> 33n
- moved R24 176.5 mm to (159.4, 174.0)
- moved R14 84.1 mm to (127.6, 102.9), turned to 270 degrees
- moved R8 81.1 mm to (66.7, 156.2), turned to 180 degrees
- moved R13 78.1 mm to (123.8, 102.9), turned to 90 degrees
- moved R11 74.9 mm to (120.0, 102.9), turned to 270 degrees
- moved R9 70.7 mm to (116.2, 102.9), turned to 90 degrees
- moved D7 65.8 mm to (135.3, 157.5)
- moved R7 65.4 mm to (66.7, 152.4), turned to 180 degrees
- moved R12 48.4 mm to (80.0, 99.7)
- moved R23 47.2 mm to (45.1, 110.5)
- moved R22 46.9 mm to (40.6, 113.7), turned to 180 degrees
- moved R21 44.6 mm to (36.2, 110.5)
- moved R34 34.8 mm to (95.2, 166.4)
- moved R17 32.7 mm to (43.8, 102.2), turned to 90 degrees
- moved R15 30.7 mm to (49.5, 102.2), turned to 270 degrees
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Connections:
- C25 pad 1: Net-(C22-Pad1) -> Net-(C1-Pad1)
- C25 pad 2: MCU_CLOCK -> Net-(C22-Pad1)
- J4 pad 2: Net-(J4-Pad2) -> GND
- J4 pad 3: GND -> EYE_GRID
- J4 pad 4: EYE_GRID -> Net-(J4-Pad4)
- K2 pad 1: +5V -> Net-(D6-Pad2)
- K2 pad 2: Net-(D6-Pad2) -> +5V
- RV1 pad 1: Net-(R34-Pad2) -> Net-(C24-Pad2)
- RV1 pad 3: Net-(C24-Pad2) -> Net-(R34-Pad2)
- U1 pad 3: Net-(U1-Pad3) -> REL_HEATER_1
- U1 pad 4: Net-(U1-Pad4) -> FLYBACK_PULSE
- U1 pad 5: Net-(U1-Pad5) -> REL_HEATER_2
- U1 pad 6: Net-(U1-Pad6) -> EYE_VOL
- U1 pad 7: Net-(U1-Pad7) -> GM_VOL
- U1 pad 8: Net-(U1-Pad8) -> GM_PULSE
- V1 pad 4: Net-(J4-Pad2) -> Net-(J4-Pad4)
Routing:
- net +5V: track 79.0 -> 315.7 mm, vias 0 -> 6
- net GND: track 166.1 -> 0.88 mm
- net EYE_VOL: track 0.00 -> 160.4 mm, vias 0 -> 2
- net GM_PULSE: track 0.00 -> 157.0 mm
- net GM_VOL: track 0.00 -> 107.9 mm, vias 0 -> 2
- net Net-(C11-Pad1): track 0.00 -> 103.3 mm
- net REL_HEATER_1: track 0.00 -> 103.3 mm, vias 0 -> 2
- net REL_HEATER_2: track 0.00 -> 101.5 mm, vias 0 -> 2
- net Net-(C5-Pad1): track 0.00 -> 86.0 mm
- net Net-(J4-Pad4): track 0.00 -> 83.5 mm
- net Net-(Q6-Pad2): track 0.00 -> 67.4 mm
- net Net-(C8-Pad1): track 0.00 -> 66.2 mm, vias 0 -> 2
- net +3V3: track 72.0 -> 136.0 mm
- net EYE_GRID: track 0.00 -> 61.8 mm
- net Net-(D2-Pad2): track 0.00 -> 57.6 mm
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- added copper zone on B.Cu, net GND
Other:
- board size 162.6 x 112.4 mm -> 160 x 112.4 mm

Commit message: Finish Geiger board.
Parts:
- removed C17: 100n, Capacitors_SMD:C_1206_HandSoldering
- removed R17: 1M, Resistors_SMD:R_1206_HandSoldering
- C13: footprint Capacitors_ThroughHole:CP_Radial_D8.0mm_P5.00mm -> Capacitors_ThroughHole:CP_Radial_D12.5mm_P5.00mm
- C14: value 1000u -> 220u; footprint Capacitors_ThroughHole:CP_Radial_D16.0mm_P7.50mm -> Capacitors_ThroughHole:CP_Radial_D12.5mm_P5.00mm
- D5, D6: footprint Diodes_ThroughHole:D_DO-41_SOD81_P10.16mm_Horizontal -> Diodes_ThroughHole:D_DO-41_SOD81_P12.70mm_Horizontal
- D7: footprint Diodes_ThroughHole:D_DO-35_SOD27_P7.62mm_Horizontal -> Diodes_ThroughHole:D_DO-35_SOD27_P10.16mm_Horizontal
- R12: footprint Resistors_SMD:R_1206_HandSoldering -> Resistors_ThroughHole:R_Axial_DIN0309_L9.0mm_D3.2mm_P12.70mm_Horizontal; moved to F.Cu
- R15: value 1M -> 2M2; footprint Resistors_SMD:R_1206_HandSoldering -> Resistors_ThroughHole:R_Axial_DIN0309_L9.0mm_D3.2mm_P12.70mm_Horizontal; moved to F.Cu
- R25, R26: footprint Resistors_ThroughHole:R_Axial_DIN0309_L9.0mm_D3.2mm_P12.70mm_Horizontal -> Resistors_ThroughHole:R_Axial_DIN0309_L9.0mm_D3.2mm_P15.24mm_Horizontal
- moved R10 75.0 mm to (156.2, 95.9)
- moved R24 72.9 mm to (154.3, 101.3), turned to 90 degrees
- moved R15 72.6 mm to (71.4, 33.0), turned to 180 degrees
- moved R19 71.2 mm to (136.8, 31.8), turned to 180 degrees
- moved D3 71.0 mm to (99.1, 39.1)
- moved R23 69.9 mm to (48.3, 40.6)
- moved R22 69.3 mm to (44.1, 44.5)
- moved R12 68.8 mm to (97.2, 33.0)
- moved R5 68.0 mm to (149.2, 87.0)
- moved R1 67.9 mm to (161.3, 109.2)
- moved R9 67.9 mm to (105.1, 35.9), turned to 270 degrees
- moved C24 67.7 mm to (81.3, 98.4)
- moved C11 67.3 mm to (46.4, 50.2)
- moved C16 67.0 mm to (69.8, 114.3)
- moved R20 66.7 mm to (140.7, 27.9)
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Connections:
- R15 pad 2: Net-(R15-Pad2) -> Net-(G1-PadA)
- U1 pad 10: DAC_CE -> DAC_CS
- U1 pad 9: DAC_CS -> DAC_CE
- V1 pad 3: Net-(K1-Pad7) -> Net-(J4-Pad4)
- V1 pad 4: Net-(J4-Pad4) -> Net-(K1-Pad7)
Routing:
- net GND: track 0.88 -> 32.0 mm, vias 0 -> 2
- net Net-(C8-Pad1): track 66.2 -> 41.9 mm, vias 2 -> 0
- net Net-(G1-PadA): track 11.0 -> 28.2 mm
- net REL_HEATER_2: track 101.5 -> 118.2 mm
- net Net-(R12-Pad2): track 28.8 -> 13.0 mm, vias 2 -> 0
- net DAC_CS: track 64.3 -> 49.8 mm
- net Net-(J4-Pad4): track 83.5 -> 73.0 mm
- net GM_VOL: track 107.9 -> 98.0 mm
- net EYE_VOL: track 160.4 -> 150.8 mm
- net GM_PULSE: track 157.0 -> 165.8 mm
- net Net-(D2-Pad2): track 57.6 -> 66.3 mm
- net DAC_CE: track 49.5 -> 56.6 mm
- net Net-(C24-Pad1): track 31.5 -> 24.5 mm
- net Net-(C19-Pad1): track 22.1 -> 15.2 mm
- net Net-(Q5-Pad2): track 39.2 -> 32.6 mm
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Other:
- rule via_min_drill: 0.3 -> 0
- board text added: "2017"
- board text added: "Michał"
- board text added: "Słomkowski"

Commit message: Small modifications of Geiger board.
Routing:
- net Net-(C8-Pad1): track 41.9 -> 44.1 mm

Commit message: Update element values on the schematic.
Parts:
- C1, C15, C27: value 33n -> 47n
- C10: value 10n -> 1n
- C20, C21: value C -> 33p
- C22: value 47p -> 150p
- C25: value 33n -> 22n
- Q2: value BC140 -> BC211
- Q3: value BC160 -> BC313
- R1: value 1k -> 1k5
- R10: value 4k7 -> 3k9
- R11, R13, R14, R21, R22, R23, R9: value 1M -> 180k
- R18, R27, R37, R38: value 47k -> 38k
- R2: value 47k -> 56k
- R20: value 330k -> 475k
- R24: value 2k2 -> 4k7
- R3: value 4k7 -> 3k3
- R39: value 10k -> 6k8
- R5: value 10 -> 1R7
Changed lines of the file:
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@@
     (links 213)
     (no_connects 0)
-    (area 15.5575 15.24 194.936786 143.035001)
+    (area 16.142499 15.824999 176.262501 128.320001)
     (thickness 1.6)
     (drawings 11)
@@
   )
   (setup
-    (last_trace_width 2.2)
+    (last_trace_width 0.25)
     (user_trace_width 0.3)
     (user_trace_width 0.3)
@@
       (effects (font (size 1 1) (thickness 0.15)))
     )
-    (fp_text value BC160 (at 2.54 5.82) (layer F.Fab)
+    (fp_text value BC313 (at 2.54 5.82) (layer F.Fab)
       (effects (font (size 1 1) (thickness 0.15)))
     )
@@
       (effects (font (size 1 1) (thickness 0.15)))
     )
-    (fp_text value BC140 (at 2.54 5.82) (layer F.Fab)
+    (fp_text value BC211 (at 2.54 5.82) (layer F.Fab)
       (effects (font (size 1 1) (thickness 0.15)))
     )
@@
       (effects (font (size 1 1) (thickness 0.15)))
     )
-    (fp_text value 4k7 (at 5.08 2.31 90) (layer F.Fab)
+    (fp_text value 3k3 (at 5.08 2.31 90) (layer F.Fab)
       (effects (font (size 1 1) (thickness 0.15)))
     )
@@
       (effects (font (size 1 1) (thickness 0.15)) (justify mirror))
     )
-    (fp_text value 10n (at 0 -2 270) (layer B.Fab)
+    (fp_text value 1n (at 0 -2 270) (layer B.Fab)
       (effects (font (size 1 1) (thickness 0.15)) (justify mirror))
     )
@@
       (effects (font (size 1 1) (thickness 0.15)))
     )
-    (fp_text value C (at 2.5 2.56 90) (layer F.Fab)
+    (fp_text value 33p (at 2.5 2.56 90) (layer F.Fab)
       (effects (font (size 1 1) (thickness 0.15)))
     )
@@
       (effects (font (size 1 1) (thickness 0.15)))
     )
-    (fp_text value C (at 2.5 2.56 90) (layer F.Fab)
+    (fp_text value 33p (at 2.5 2.56 90) (layer F.Fab)
       (effects (font (size 1 1) (thickness 0.15)))
     )
@@
       (effects (font (size 1 1) (thickness 0.15)))
     )
-    (fp_text value 47p (at 2.5 2.56 90) (layer F.Fab)
+    (fp_text value 150p (at 2.5 2.56 90) (layer F.Fab)
       (effects (font (size 1 1) (thickness 0.15)))
     )
@@
       (effects (font (size 1 1) (thickness 0.15)))
     )
-    (fp_text value 33n (at 2.5 2.56 180) (layer F.Fab)
+    (fp_text value 22n (at 2.5 2.56 180) (layer F.Fab)
       (effects (font (size 1 1) (thickness 0.15)))
     )
@@
       (effects (font (size 1 1) (thickness 0.15)) (justify mirror))
     )
-    (fp_text value 1M (at 0 -1.9 270) (layer B.Fab)
+    (fp_text value 180k (at 0 -1.9 270) (layer B.Fab)
       (effects (font (size 1 1) (thickness 0.15)) (justify mirror))
     )
@@
       (effects (font (size 1 1) (thickness 0.15)) (justify mirror))
     )
-    (fp_text value 4k7 (at 0 -1.9) (layer B.Fab)
+    (fp_text value 3k9 (at 0 -1.9) (layer B.Fab)
       (effects (font (size 1 1) (thickness 0.15)) (justify mirror))
     )
@@
       (effects (font (size 1 1) (thickness 0.15)) (justify mirror))
     )
-    (fp_text value 1M (at 0 -1.9 270) (layer B.Fab)
+    (fp_text value 180k (at 0 -1.9 270) (layer B.Fab)
       (effects (font (size 1 1) (thickness 0.15)) (justify mirror))
     )
@@
       (effects (font (size 1 1) (thickness 0.15)) (justify mirror))
     )
-    (fp_text value 1M (at 0 -1.9 90) (layer B.Fab)
+    (fp_text value 180k (at 0 -1.9 90) (layer B.Fab)
       (effects (font (size 1 1) (thickness 0.15)) (justify mirror))
     )
@@
       (effects (font (size 1 1) (thickness 0.15)) (justify mirror))
     )
-    (fp_text value 1M (at 0 -1.9 270) (layer B.Fab)
+    (fp_text value 180k (at 0 -1.9 270) (layer B.Fab)
       (effects (font (size 1 1) (thickness 0.15)) (justify mirror))
     )
@@
       (effects (font (size 1 1) (thickness 0.15)) (justify mirror))
     )
-    (fp_text value 47k (at 0 -1.9 270) (layer B.Fab)
+    (fp_text value 38k (at 0 -1.9 270) (layer B.Fab)
       (effects (font (size 1 1) (thickness 0.15)) (justify mirror))
     )
@@
       (effects (font (size 1 1) (thickness 0.15)) (justify mirror))
     )
-    (fp_text value 330k (at 0 -1.9) (layer B.Fab)
+    (fp_text value 475k (at 0 -1.9) (layer B.Fab)
       (effects (font (size 1 1) (thickness 0.15)) (justify mirror))
     )
@@
       (effects (font (size 1 1) (thickness 0.15)) (justify mirror))
     )
-    (fp_text value 1M (at 0 -1.9 90) (layer B.Fab)
+    (fp_text value 180k (at 0 -1.9 90) (layer B.Fab)
       (effects (font (size 1 1) (thickness 0.15)) (justify mirror))
     )
@@
       (effects (font (size 1 1) (thickness 0.15)) (justify mirror))
     )
-    (fp_text value 1M (at 0 -1.9 180) (layer B.Fab)
+    (fp_text value 180k (at 0 -1.9 180) (layer B.Fab)
       (effects (font (size 1 1) (thickness 0.15)) (justify mirror))
     )
@@
       (effects (font (size 1 1) (thickness 0.15)) (justify mirror))
     )
-    (fp_text value 1M (at 0 -1.9) (layer B.Fab)
+    (fp_text value 180k (at 0 -1.9) (layer B.Fab)
       (effects (font (size 1 1) (thickness 0.15)) (justify mirror))
     )
@@
       (effects (font (size 1 1) (thickness 0.15)) (justify mirror))
     )
-    (fp_text value 2k2 (at 0 -1.9 90) (layer B.Fab)
+    (fp_text value 4k7 (at 0 -1.9 90) (layer B.Fab)
       (effects (font (size 1 1) (thickness 0.15)) (justify mirror))
     )
@@
       (effects (font (size 1 1) (thickness 0.15)) (justify mirror))
     )
-    (fp_text value 47k (at 0 -1.9 270) (layer B.Fab)
+    (fp_text value 38k (at 0 -1.9 270) (layer B.Fab)
       (effects (font (size 1 1) (thickness 0.15)) (justify mirror))
     )
@@
       (effects (font (size 1 1) (thickness 0.15)) (justify mirror))
     )
-    (fp_text value 47k (at 0 -1.9 270) (layer B.Fab)
+    (fp_text value 38k (at 0 -1.9 270) (layer B.Fab)
       (effects (font (size 1 1) (thickness 0.15)) (justify mirror))
     )
@@
       (effects (font (size 1 1) (thickness 0.15)) (justify mirror))
     )
-    (fp_text value 47k (at 0 -1.9 90) (layer B.Fab)
+    (fp_text value 38k (at 0 -1.9 90) (layer B.Fab)
       (effects (font (size 1 1) (thickness 0.15)) (justify mirror))
     )
@@
       (effects (font (size 1 1) (thickness 0.15)))
     )
-    (fp_text value 1k (at 5.08 2.31 90) (layer F.Fab)
+    (fp_text value 1k5 (at 5.08 2.31 90) (layer F.Fab)
       (effects (font (size 1 1) (thickness 0.15)))
     )
@@
       (effects (font (size 1 1) (thickness 0.15)))
     )
-    (fp_text value 47k (at 5.08 2.31 90) (layer F.Fab)
+    (fp_text value 56k (at 5.08 2.31 90) (layer F.Fab)
       (effects (font (size 1 1) (thickness 0.15)))
     )
@@
       (effects (font (size 1 1) (thickness 0.15)))
     )
-    (fp_text value 10 (at 5.08 2.31 90) (layer F.Fab)
+    (fp_text value 1R7 (at 5.08 2.31 90) (layer F.Fab)
       (effects (font (size 1 1) (thickness 0.15)))
     )
@@
       (effects (font (size 1 1) (thickness 0.15)))
     )
-    (fp_text value 10k (at 6.35 2.66 180) (layer F.Fab)
+    (fp_text value 6k8 (at 6.35 2.66 180) (layer F.Fab)
       (effects (font (size 1 1) (thickness 0.15)))
     )
@@
       (effects (font (size 1 1) (thickness 0.15)))
     )
-    (fp_text value 33n (at 2.5 2.56 270) (layer F.Fab)
+    (fp_text value 47n (at 2.5 2.56 270) (layer F.Fab)
       (effects (font (size 1 1) (thickness 0.15)))
     )
@@
       (effects (font (size 1 1) (thickness 0.15)))
     )
-    (fp_text value 33n (at 2.5 2.56 180) (layer F.Fab)
+    (fp_text value 47n (at 2.5 2.56 180) (layer F.Fab)
       (effects (font (size 1 1) (thickness 0.15)))
     )
@@
       (effects (font (size 1 1) (thickness 0.15)))
     )
-    (fp_text value 33n (at 2.5 2.56) (layer F.Fab)
+    (fp_text value 47n (at 2.5 2.56) (layer F.Fab)
       (effects (font (size 1 1) (thickness 0.15)))
     )
