File: pcb/clock-display/clock-display.sch (KiCad schematic (older format))
At the start: 36 parts, among them CON1 AVR-ISP-10, IC1 ATTINY26-S, IC2 TD62C950RF, IC3 RFM83C-433S, K1 V23079, K2 V23079, P1 CONN_02X05, P2 CONN_01X02, P3 CONN_01X04, P4 CONN_01X04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

Commit message: Update all Kicad files to Kicad 5.
Parts:
- C1, C6: symbol CP -> clock-display-rescue:CP
- C2, C3, C4, C5: symbol C_Small -> clock-display-rescue:C_Small
- CON1: symbol AVR-ISP-10 -> clock-display-rescue:AVR-ISP-10
- D1, D2: symbol D -> clock-display-rescue:D
- IC1: symbol ATTINY26-S -> clock-display-rescue:ATTINY26-S
- IC2: symbol TD62C950RF -> TD62C950RF:TD62C950RF
- IC3: symbol RFM83C-433S -> RFM83C-433S:RFM83C-433S
- K1, K2: symbol V23079 -> V23079-monostable:V23079
- P1: symbol CONN_02X05 -> clock-display-rescue:CONN_02X05
- P2, P8: symbol CONN_01X02 -> clock-display-rescue:CONN_01X02
- P3, P4, P5, P6, P7: symbol CONN_01X04 -> clock-display-rescue:CONN_01X04
- Q1, Q2: symbol BC849 -> clock-display-rescue:BC849
- R1, R10, R11, R2, R3, R4, R5, R6, R7, R8, R9: symbol R -> clock-display-rescue:R
- SV1: symbol 5-LT-02M -> futaba-vfd:5-LT-02M
Connections:
- wire segments 220 -> 241
