File: pcb/clock-display/clock-display.kicad_pcb (KiCad board)
At the start: 2 copper layers, 108.5 x 54.6 mm, 43 parts, among them CON1 AVR-ISP-10, IC1 ATTINY26-S, IC2 TD62C950RF, IC3 RFM83C-433S, K1 V23079, K2 V23079, P1 CONN_02X05, P2 CONN_01X02, P3 CONN_01X04, P4 CONN_01X04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

Commit message: Fix analog gauge clicking.
Other:
- net class Default removed

Commit message: Migrate to KiCAD 9.
Parts:
- R3, R4: value 220 -> 5R1
Connections:
- CON1 pad 3: (no net) -> unconnected-(CON1-Pad3)
- IC1 pad 13: (no net) -> unconnected-(IC1-(ADC4)PA5-Pad13)
- IC1 pad 20: (no net) -> unconnected-(IC1-(ADC0)PA0-Pad20)
- IC1 pad 7: (no net) -> unconnected-(IC1-(ADC7/XTAL1)PB4-Pad7)
- IC1 pad 8: (no net) -> unconnected-(IC1-(ADC8/XTAL2)PB5-Pad8)
- IC2 pad 16: (no net) -> unconnected-(IC2-OUT25-Pad16)
- IC2 pad 17: (no net) -> unconnected-(IC2-OUT24-Pad17)
- IC2 pad 18: (no net) -> unconnected-(IC2-OUT23-Pad18)
- IC2 pad 19: (no net) -> unconnected-(IC2-OUT22-Pad19)
- IC2 pad 20: (no net) -> unconnected-(IC2-OUT21-Pad20)
- IC2 pad 29: (no net) -> unconnected-(IC2-S-OUT-Pad29)
- IC2 pad 41: (no net) -> unconnected-(IC2-OUT20-Pad41)
- IC2 pad 42: (no net) -> unconnected-(IC2-OUT19-Pad42)
- IC2 pad 43: (no net) -> unconnected-(IC2-OUT18-Pad43)
- IC2 pad 44: (no net) -> unconnected-(IC2-OUT17-Pad44)
- IC2 pad 45: (no net) -> unconnected-(IC2-OUT16-Pad45)
- IC3 pad 3: (no net) -> unconnected-(IC3-SHUT-Pad3)
- P1 pad 10: (no net) -> unconnected-(P1-P10-Pad10)
- P1 pad 4: (no net) -> unconnected-(P1-P4-Pad4)
- P1 pad 6: (no net) -> unconnected-(P1-P6-Pad6)
- P1 pad 7: (no net) -> unconnected-(P1-P7-Pad7)
- P3 pad 3: (no net) -> unconnected-(P3-P3-Pad3)
- P4 pad 4: (no net) -> unconnected-(P4-P4-Pad4)
- P5 pad 3: (no net) -> unconnected-(P5-P3-Pad3)
- P6 pad 2: (no net) -> unconnected-(P6-P2-Pad2)
