File: pcb/front-display/front-display.sch (KiCad schematic (older format))
At the start: 57 parts, among them CON1 AVR-ISP-10, IC1 ATMEGA88A-A, IC2 TD62C950RF, IC3 TD62C950RF, J1 HEADER_5, P1 CONN_02X05, P2 CONN_01X03, P3 CONN_01X02, P4 CONN_01X04, P5 CONN_01X02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

Commit message: Move PCB projects to new names.
Parts:
- L1: symbol INDUCTOR-RESCUE-vfd-display-front -> INDUCTOR-RESCUE-front-display
- U3: symbol LM1117-3.3-RESCUE-vfd-display-front -> LM1117-3.3-RESCUE-front-display
Changed lines of the file:
@@
 EESchema Schematic File Version 2
-LIBS:vfd-display-front-rescue
+LIBS:front-display-rescue
 LIBS:power
 LIBS:device
@@
 LIBS:futaba-vfd
 LIBS:TD62C950RF
-LIBS:vfd-display-front-cache
+LIBS:front-display-cache
 EELAYER 25 0
 EELAYER END
@@
 $EndComp
 $Comp
-L INDUCTOR-RESCUE-vfd-display-front L1
+L INDUCTOR-RESCUE-front-display L1
 U 1 1 578034BB
 P 12550 8100
@@
 $EndComp
 $Comp
-L LM1117-3.3-RESCUE-vfd-display-front U3
+L LM1117-3.3-RESCUE-front-display U3
 U 1 1 578CCB5D
 P 14400 8100

Commit message: Update all Kicad files to Kicad 5.
Parts:
- C1, C10, C11, C12, C14, C15, C16, C2, C6, C7, C8, C9: symbol C_Small -> front-display-rescue:C_Small
- C13, C17, C19, C3, C4, C5: symbol CP -> front-display-rescue:CP
- CON1: symbol AVR-ISP-10 -> front-display-rescue:AVR-ISP-10
- D1, D2, D3, D4, D5, D6: symbol DIODE -> front-display-rescue:DIODE
- D7: symbol SCHOTTKY -> front-display-rescue:SCHOTTKY
- IC1: symbol ATMEGA88A-A -> front-display-rescue:ATMEGA88A-A
- IC2, IC3: symbol TD62C950RF -> front-display-rescue:TD62C950RF
- J1: symbol HEADER_5 -> front-display-rescue:HEADER_5
- L1: symbol INDUCTOR-RESCUE-front-display -> front-display-rescue:INDUCTOR-RESCUE-front-display
- P1: symbol CONN_02X05 -> front-display-rescue:CONN_02X05
- P2: symbol CONN_01X03 -> front-display-rescue:CONN_01X03
- P3, P5, P6: symbol CONN_01X02 -> front-display-rescue:CONN_01X02
- P4: symbol CONN_01X04 -> front-display-rescue:CONN_01X04
- Q1: symbol BC849 -> front-display-rescue:BC849
- R1, R10, R11, R12, R13, R14, R2, R3, R4, R5, R6, R7, R8, R9: symbol R -> front-display-rescue:R
- SV1: symbol 202-MD-08GK -> front-display-rescue:202-MD-08GK
- U1: symbol LM2596 -> front-display-rescue:LM2596
- U2: symbol ESP-12E -> front-display-rescue:ESP-12E
- U3: symbol LM1117-3.3-RESCUE-front-display -> front-display-rescue:LM1117-3.3-RESCUE-front-display
- Y1: symbol Crystal_Small -> front-display-rescue:Crystal_Small
