File: pcb/front-display/front-display.kicad_pcb (KiCad board)
At the start: 2 copper layers, 201.9 x 54.6 mm, 61 parts, among them CON1 AVR-ISP-10, IC1 ATMEGA88A-A, IC2 TD62C950RF, IC3 TD62C950RF, J1 HEADER_5, P1 CONN_02X05, P2 CONN_01X03, P3 CONN_01X02, P4 CONN_01X04, P5 CONN_01X02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

Commit message: Migrate to KiCAD 9.
Parts:
- R8, R9: value 100 -> 5R1
Connections:
- CON1 pad 3: (no net) -> unconnected-(CON1-Pad3)
- IC1 pad 19: (no net) -> unconnected-(IC1-ADC6-Pad19)
- IC1 pad 2: (no net) -> unconnected-(IC1-(PCINT20/XCK/T0)PD4-Pad2)
- IC1 pad 20: (no net) -> unconnected-(IC1-AREF-Pad20)
- IC1 pad 22: (no net) -> unconnected-(IC1-ADC7-Pad22)
- IC1 pad 23: (no net) -> unconnected-(IC1-(PCINT8/ADC0)PC0-Pad23)
- IC1 pad 24: (no net) -> unconnected-(IC1-(PCINT9/ADC1)PC1-Pad24)
- IC1 pad 25: (no net) -> unconnected-(IC1-(PCINT10/ADC2)PC2-Pad25)
- IC1 pad 26: (no net) -> unconnected-(IC1-(PCINT11/ADC3)PC3-Pad26)
- IC1 pad 30: (no net) -> unconnected-(IC1-(PCINT16/RXD)PD0-Pad30)
- IC2 pad 1: (no net) -> unconnected-(IC2-OUT40-Pad1)
- IC2 pad 2: (no net) -> unconnected-(IC2-OUT39-Pad2)
- IC3 pad 29: (no net) -> unconnected-(IC3-S-OUT-Pad29)
- IC3 pad 57: (no net) -> unconnected-(IC3-OUT4-Pad57)
- IC3 pad 58: (no net) -> unconnected-(IC3-OUT3-Pad58)
- P1 pad 4: (no net) -> unconnected-(P1-P4-Pad4)
- P1 pad 6: (no net) -> unconnected-(P1-P6-Pad6)
- P1 pad 7: (no net) -> unconnected-(P1-P7-Pad7)
- U2 pad 10: (no net) -> unconnected-(U2-MISO-Pad10)
- U2 pad 11: (no net) -> unconnected-(U2-GPIO9-Pad11)
- U2 pad 12: (no net) -> unconnected-(U2-GPIO10-Pad12)
- U2 pad 13: (no net) -> unconnected-(U2-MOSI-Pad13)
- U2 pad 14: (no net) -> unconnected-(U2-SCLK-Pad14)
- U2 pad 17: (no net) -> unconnected-(U2-GPIO2-Pad17)
- U2 pad 2: (no net) -> unconnected-(U2-ADC-Pad2)
- U2 pad 4: (no net) -> unconnected-(U2-GPIO16-Pad4)
- U2 pad 5: (no net) -> unconnected-(U2-GPIO14-Pad5)
- U2 pad 7: (no net) -> unconnected-(U2-GPIO13-Pad7)
- U2 pad 9: (no net) -> unconnected-(U2-CS0-Pad9)
Other:
- net class Default removed
