File: pcb/rotary-encoder/rotary-encoder.kicad_pcb (KiCad board)
At the start: 2 copper layers, 10 parts, among them J1 Conn_01x05, SW1 EC11

Commit message: Rotary encoder board.
Parts:
- C1, C2, C3, R1, R2, R3, R4, R5: moved to B.Cu
- moved SW1 62.5 mm to (39.9, 99.2)
- moved R2 57.3 mm to (46.8, 102.5), turned to 180 degrees
- moved C3 55.9 mm to (51.2, 102.7), turned to -90 degrees
- moved R3 53.8 mm to (44.9, 99.7), turned to 180 degrees
- moved R1 51.1 mm to (53.1, 95.9)
- moved R5 49.9 mm to (39.9, 94.8), turned to -90 degrees
- moved R4 49.5 mm to (43.0, 94.8), turned to 90 degrees
- moved C1 47.8 mm to (61.2, 96.6)
- moved C2 47.8 mm to (61.2, 100.0)
- moved J1 44.0 mm to (48.5, 92.4), turned to 90 degrees
Connections:
- C1 pad 1: Net-(J1-Pin_2) -> Net-(J1-Pin_4)
- R1 pad 2: Net-(J1-Pin_4) -> Net-(J1-Pin_2)
- R5 pad 1: Net-(J1-Pin_2) -> Net-(J1-Pin_4)
- SW1 pad S1: GND -> Net-(J1-Pin_2)
- SW1 pad S2: Net-(J1-Pin_4) -> GND
Routing:
- net Net-(J1-Pin_4): track 0.00 -> 26.7 mm
- net Net-(J1-Pin_3): track 0.00 -> 24.7 mm
- net VCC: track 0.00 -> 17.8 mm
- net Net-(R2-Pad2): track 0.00 -> 13.1 mm
- net Net-(J1-Pin_2): track 0.00 -> 8.74 mm
- net Net-(R3-Pad2): track 0.00 -> 6.49 mm
- net (no net): vias 0 -> 4
- added copper zone on B.Cu, net GND
Other:
- board outline added: 51 x 27 mm
- board text added: "2025"
- board text added: "Octoglow"
- board text added: "slomkowski.eu"
